File: PCB/Macropad.kicad_pcb (KiCad board)
At the start: 2 copper layers, 58 x 85.9 mm, 9 parts, among them SW1 SW_Push, SW2 SW_Push, SW3 SW_Push, SW4 SW_Push, SW5 SW_Push, SW6 SW_Push, U1 XIAO-RP2040-DIP

Commit message: edited
edited
Parts:
- added D3: SK6812MINI, LED_SMD:LED_SK6812MINI_PLCC4_3.5x3.5mm_P1.75mm, F.Cu at (138.3, 118.5)
- added D4: SK6812MINI, LED_SMD:LED_SK6812MINI_PLCC4_3.5x3.5mm_P1.75mm, F.Cu at (187.0, 117.8)
- moved D2 5.52 mm to (182.8, 48.9)
- moved D1 5.04 mm to (141.8, 48.9)
Connections:
- D2 pad 1: unconnected-(D2-DOUT-Pad1) -> Net-(D2-DOUT)
Routing:
- net +5V: track 34.9 -> 177.0 mm, vias 0 -> 2
- net Net-(D2-DOUT): track 0.00 -> 103.1 mm
- net Net-(D3-DOUT): track 0.00 -> 56.9 mm
- net GND: track 149.3 -> 204.3 mm, vias 0 -> 5
- net Net-(D1-DOUT): track 43.0 -> 54.2 mm
- net Net-(U1-GPIO2/SCK): track 53.6 -> 60.3 mm
- net Net-(D1-DIN): track 7.48 -> 12.1 mm
Other:
- board text added: "-_-_-_-_-_-_-_-_-_-_-_-_-_-_-_-_-_-_-_-"
- board text added: "_-_-_-_-_-_-_-_-_-_-_-_-_-_-_-"

Commit message: submit
submit
Parts:
- added G***: LOGO, LOGO, F.Cu at (187.3, 93.7)
- added G***: LOGO, LOGO, F.Cu at (187.3, 74.2)
Other:
- board text removed: "-_-_-_-_-_-_-_-_-_-_-_-_-_-_-_-_-_-_-_-"
- board text removed: "_-_-_-_-_-_-_-_-_-_-_-_-_-_-_-"

Commit message: submit
Parts:
- added SW7: RotaryEncoder, Rotary_Encoder:RotaryEncoder_Alps_EC11E_Vertical_H20mm, F.Cu at (144.9, 126.5)
- added SW8: RotaryEncoder, Rotary_Encoder:RotaryEncoder_Alps_EC11E_Vertical_H20mm, F.Cu at (165.9, 126.5)
Connections:
- U1 pad 1: unconnected-(U1-GPIO26/ADC0/A0-Pad1) -> Net-(U1-GPIO26/ADC0/A0)
- U1 pad 2: unconnected-(U1-GPIO27/ADC1/A1-Pad2) -> Net-(U1-GPIO27/ADC1/A1)
- U1 pad 3: unconnected-(U1-GPIO28/ADC2/A2-Pad3) -> Net-(U1-GPIO28/ADC2/A2)
- U1 pad 4: unconnected-(U1-GPIO29/ADC3/A3-Pad4) -> Net-(U1-GPIO29/ADC3/A3)
Routing:
- net Net-(U1-GPIO29/ADC3/A3): track 0.00 -> 121.9 mm
- net Net-(U1-GPIO26/ADC0/A0): track 0.00 -> 120.2 mm
- net Net-(U1-GPIO27/ADC1/A1): track 0.00 -> 119.7 mm
- net Net-(U1-GPIO28/ADC2/A2): track 0.00 -> 87.5 mm
- net GND: track 204.3 -> 255.6 mm, vias 5 -> 7
Other:
- board size 58 x 85.9 mm -> 58 x 98.9 mm
